Commit message: Changed the wheel collision box to proper 8 mm instead of 80 mm, added the collisions, mass and inerta

File: install/ias0220_250620/share/ias0220_250620/urdf/differential_robot.urdf (robot description, URDF)
Before this commit: robot The_IAS_robot, 5 links, 4 joints
Links:
- link base_link: mass None -> ${BASE_MASS}
- link head_link: mass None -> ${HEAD_MASS}
- link passive_wheel_holder_link: mass None -> ${WHEEL_HOLDER_MASS}
- link passive_wheel_link: mass None -> ${PASSIVE_WHEEL_MASS}
