Commit message: Started the task 6.2, created a launch file and also started creating the camera for the robot

File: install/ias0220_250620/share/ias0220_250620/urdf/differential_robot_simu_task4_part2.urdf (robot description, URDF)
Before this commit: robot The_IAS_robot, 5 links, 4 joints
Links:
- added link camera_link; collision box size=${CAMERA_SIDE_SIZE} ${CAMERA_SIDE_SIZE} ${CAMERA_SIDE_SIZE}; visual box size=${CAMERA_SIDE_SIZE} ${CAMERA_SIDE_SIZE} ${CAMERA_SIDE_SIZE}
Joints:
- added joint camera_joint: type fixed, parent head_link, child camera_link, origin xyz=0 0 ${HEAD_SIDE_SIZE/2 + CAMERA_SIDE_SIZE/2} rpy=0 0 0, axis 0 1 0
