Commit message: Renamed some links according to the exercise

File: src/ias0220_250620/urdf/differential_robot.urdf (robot description, URDF)
Before this commit: robot The_IAS_robot, 5 links, 4 joints
Links:
- removed link passive_wheel_holder_link
- removed link passive_wheel_link
- added link passive_wheel, mass ${PASSIVE_WHEEL_MASS}; collision sphere radius=${SUPPORT_WIDTH/2}; visual sphere radius=${SUPPORT_WIDTH/2}
- added link passive_wheel_holder, mass ${WHEEL_HOLDER_MASS}; collision box size=${SUPPORT_WIDTH} ${SUPPORT_WIDTH} ${WHEEL_HOLDER_HEIGHT}; visual box size=${SUPPORT_WIDTH} ${SUPPORT_WIDTH} ${WHEEL_HOLDER_HEIGHT}
Joints:
- joint head_to_support_base: child passive_wheel_holder_link -> passive_wheel_holder
- joint passive_wheel_holder_to_wheel: child passive_wheel_link -> passive_wheel; parent passive_wheel_holder_link -> passive_wheel_holder
