Commit message: Completed the Task 6.2, during which I learned to create an object recognition node based on the color of the object (opencv)

File: src/ias0220_250620/urdf/differential_robot_simu_task4_part2.urdf (robot description, URDF)
Before this commit: robot The_IAS_robot, 6 links, 5 joints
Links:
- link camera_link: geometry collision box size=${CAMERA_SIDE_SIZE*2} ${CAMERA_SIDE_SIZE} ${CAMERA_SIDE_SIZ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; visual box size=${CAMERA_SIDE_SIZE*2} ${CAMERA_SIDE_SIZE} ${CAMERA_SIDE_SIZ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
